Commit message: uf850: make the xarm_gripper physics-grasp-capable under Gazebo Harmonic
Five small, independent changes needed to grasp an object with real physics
in gz-sim 8 + gz_ros2_control, found while bringing up a contact-gated
detachable-joint grasp on the uf850 cell.

* xarm_gripper.urdf.xacro — give `drive_joint` <dynamics>. It is the only
  joint in the arm with none (every arm joint has damping 3.4-16.6 /
  friction 1.1-12.1). Undamped it hunts around its setpoint by ~9e-4 rad,
  and MoveIt Task Constructor's Connect stage drops any goal whose joints
  outside the planned group differ by more than a hardcoded 1e-4
  ("Deviation in joint drive_joint"), so a pick becomes intermittently
  unplannable. A real gripper's gearbox and leadscrew are heavily damped.

* xarm_gripper.ros2_control.xacro — initial_value 0.02 on the position
  state interface. `drive_joint`'s lower limit IS 0, so starting the sim
  on that hard stop lets the solver slip the measured position a fraction
  of a milliradian negative; MoveIt/MTC then see an out-of-bounds start
  state and every gripper MoveTo fails with "Start state is out of
  bounds!" before the robot has moved. Ignored by the non-sim plugins.

* xarm_gripper_macro.xacro / xarm_device_macro.xacro — new
  `add_mimic_joint_plugin` parameter (default true, so the stock examples
  are unchanged). On Gazebo Harmonic the mimic plugin is redundant:
  sdformat14 converts each URDF <mimic> into an SDF <axis><mimic>
  constraint that gz-physics enforces directly (bullet-featherstone
  SetMimicConstraintFeature), and the fingers follow drive_joint with the
  plugin absent. It is also unsafe — GazeboMimicJointPlugin::PostUpdate
  writes a JointForceCmd component through a const ECM and intermittently
  segfaults gz-sim inside EntityComponentManager::CreateComponent.

* xarm_moveit_config/config/uf850{,_gripper}/gz_controllers.yaml — a
  MoveIt->controller routing table for the gz_ros2_control path:
  FollowJointTrajectory for the arm AND the gripper. controllers.yaml
  routes the gripper to the firmware's GripperCommand action, which only
  exists on real hardware, and borrowing fake_controllers.yaml would rely
  on its names coinciding by accident.

Co-Authored-By: Claude Opus 5 (1M context) <noreply@anthropic.com>

File: xarm_description/urdf/gripper/xarm_gripper.ros2_control.xacro (robot description, xacro)
@@ -14,5 +14,14 @@
           <param name="max">3.14</param>
         </command_interface>
-        <state_interface name="position"/>
+        <!-- initial_value 0.02, not the implicit 0: `drive_joint`'s lower joint limit IS 0, so
+             starting the sim at 0 parks the joint on its hard stop and a physics engine jitters it a
+             fraction of a milliradian NEGATIVE. MoveIt/MTC then see an out-of-bounds start state and
+             every gripper MoveTo fails with "Start state is out of bounds!" before the robot has
+             done anything. 0.02 rad is ~1 mm of jaw travel and matches the SRDF 'open' pose, so the
+             gripper simply boots where 'open' already puts it. The non-sim hardware plugins read a
+             real encoder and ignore this. -->
+        <state_interface name="position">
+          <param name="initial_value">0.02</param>
+        </state_interface>
         <state_interface name="velocity"/>
         <!-- <state_interface name="effort"/> -->

File: xarm_description/urdf/gripper/xarm_gripper.urdf.xacro (robot description, xacro)
@@ -57,4 +57,11 @@
       <axis xyz="1 0 0" />
       <limit lower="0" upper="0.85" effort="50" velocity="2" />
+      <!-- The only actuated gripper joint, and the only one in the arm's URDF with no <dynamics>
+           (every arm joint has damping 3.4-16.6 / friction 1.1-12.1). Undamped it HUNTS around its
+           setpoint in Gazebo by ~9e-4 rad, and MTC's Connect drops any goal whose joints outside the
+           planned group differ by more than a hardcoded 1e-4 — so an undamped gripper makes Pick
+           intermittently unplannable ("Deviation in joint drive_joint"). A real gripper's gearbox
+           and leadscrew are heavily damped, so modelling that is also just more truthful. -->
+      <dynamics damping="1.0" friction="0.5" />
     </joint>
     <link name="${prefix}left_finger">

File: xarm_description/urdf/gripper/xarm_gripper_macro.xacro (robot description, xacro)
@@ -7,5 +7,6 @@
   <xacro:include filename="$(find xarm_description)/urdf/gripper/xarm_gripper.gazebo.xacro" />
   <xacro:macro name="xarm_gripper_macro" params="prefix:='' attach_to:='' ns:='xarm' attach_xyz:='0 0 0' attach_rpy:='0 0 0'
-    ros2_control_plugin:='uf_robot_hardware/UFRobotFakeSystemHardware' dof:=7 hard_interface:='PositionJointInterface' gripper_version:='G1'"> ">
+    ros2_control_plugin:='uf_robot_hardware/UFRobotFakeSystemHardware' dof:=7 hard_interface:='PositionJointInterface' gripper_version:='G1'
+    add_mimic_joint_plugin:=true"> ">
     <xacro:if value="${is_ros2 and ros2_control_plugin != 'uf_robot_hardware/UFRobotSystemHardware'}">
       <xacro:xarm_gripper_ros2_control prefix="${prefix}" ros2_control_plugin="${ros2_control_plugin}" />
@@ -17,5 +18,14 @@
       <xacro:xarm_gazebo_grasp_fix prefix="${prefix}" palm_link="${prefix}link${dof}" />
     </xacro:if>
-    <!-- mimic_joint_plugin has to be installed: -->
+    <!-- mimic_joint_plugin has to be installed.
+         `add_mimic_joint_plugin:=false` skips it: on Gazebo Harmonic it is REDUNDANT and UNSAFE.
+         Redundant because sdformat14 converts each URDF <mimic> into an SDF <axis><mimic> constraint
+         that gz-physics enforces directly (bullet-featherstone SetMimicConstraintFeature) — the
+         finger joints follow drive_joint with the plugin absent. Unsafe because
+         GazeboMimicJointPlugin::PostUpdate writes a JointForceCmd component through a const ECM,
+         which intermittently segfaults gz-sim inside EntityComponentManager::CreateComponent
+         (observed while bringing up the uf850_cell physics grasp). Default stays true so the stock
+         examples are unchanged. -->
+    <xacro:if value="${add_mimic_joint_plugin}">
     <xacro:mimic_joint_plugin_gazebo name_prefix="${prefix}left_finger_joint"
       following_joint="${prefix}drive_joint" mimic_joint="${prefix}left_finger_joint"
@@ -33,4 +43,5 @@
       following_joint="${prefix}drive_joint" mimic_joint="${prefix}right_inner_knuckle_joint"
       has_pid="${is_ros2}" multiplier="1.0" max_effort="10.0" ros2_control_plugin="${ros2_control_plugin}"/>
+    </xacro:if>
   </xacro:macro>
 </robot>

File: xarm_description/urdf/xarm_device_macro.xacro (robot description, xacro)
@@ -43,4 +43,5 @@
     kinematics_suffix:=''
     gripper_version:='G1'
+    add_mimic_joint_plugin:=true
     "
     >
@@ -245,5 +246,5 @@
         <xacro:xarm_gripper_macro prefix="${prefix}" attach_to="${prefix}link_eef"
           ros2_control_plugin="${ros2_control_plugin}" dof="${dof}" hard_interface="${hard_interface}"
-          gripper_version="${gripper_version}" />
+          gripper_version="${gripper_version}" add_mimic_joint_plugin="${add_mimic_joint_plugin}" />
       </xacro:unless>
     </xacro:if>
