Commit message: uf850: never park the gripper on its hard stop
`drive_joint`'s lower joint limit IS 0, and the SRDF "open" group state was
also 0 — so the fully-open pose parked the joint against a hard stop. A
physics engine does not settle exactly on a hard stop: gz/bullet-featherstone
left the measured position a fraction of a milliradian NEGATIVE (-4.0e-04
observed). MoveIt and MTC then judge the whole robot state out of bounds, and
every subsequent gripper MoveTo fails with "Start state is out of bounds!" —
so after the first ReturnHome the arm could never pick again.

* _uf850_macro.srdf.xacro — "open" 0 -> 0.02 rad (~1 mm of jaw travel). The
  gripper is still fully open for anything the cell handles, and the joint no
  longer rests against its limit.

* xarm_gripper.urdf.xacro — 5 mrad of slack below zero on drive_joint AND its
  five <mimic> followers, as defence in depth. MTC validates every joint in
  the state, so widening only the driven joint would leave the followers out
  of bounds. This does not change where the jaws actually stop, which is set
  by mesh contact.

Co-Authored-By: Claude Opus 5 (1M context) <noreply@anthropic.com>

File: xarm_description/urdf/gripper/xarm_gripper.urdf.xacro (robot description, xacro)
@@ -1,4 +1,14 @@
 <?xml version="1.0"?>
 <robot xmlns:xacro="http://ros.org/wiki/xacro" name="xarm_gripper">
+  <!-- The gripper's fully-open pose IS its lower joint limit (SRDF group_state "open" = 0), so the
+       jaws come to rest against a hard stop. A physics engine does not stop exactly on a hard stop:
+       gz/bullet-featherstone settles a fraction of a milliradian past it (-4.0e-04 measured). MoveIt
+       and MTC then judge the whole robot state OUT OF BOUNDS, and every subsequent gripper MoveTo
+       fails with "Start state is out of bounds!" — so after the first ReturnHome the arm can never
+       pick again. Giving each gripper joint 5 mrad (~0.25 mm of jaw) of slack below zero absorbs
+       that without changing where the jaws actually stop, which is set by mesh contact, not by this
+       number. Applies to drive_joint AND its five <mimic> followers: MTC validates every joint in
+       the state, so widening only the driven one leaves the followers out of bounds. -->
+  <xacro:property name="gripper_eps" value="-0.005"/>
   <xacro:macro name="xarm_gripper_urdf" params="prefix:='' attach_to:='' attach_xyz:='0 0 0' attach_rpy:='0 0 0' gripper_version:='G1' ">
     <xacro:property name="name_suffix" value=""/>
@@ -56,5 +66,5 @@
       <child link="${prefix}left_outer_knuckle" />
       <axis xyz="1 0 0" />
-      <limit lower="0" upper="0.85" effort="50" velocity="2" />
+      <limit lower="${gripper_eps}" upper="0.85" effort="50" velocity="2" />
       <!-- The only actuated gripper joint, and the only one in the arm's URDF with no <dynamics>
            (every arm joint has damping 3.4-16.6 / friction 1.1-12.1). Undamped it HUNTS around its
@@ -88,5 +98,5 @@
       <child link="${prefix}left_finger" />
       <axis xyz="-1 0 0" />
-      <limit lower="0" upper="0.85" effort="50" velocity="2" />
+      <limit lower="${gripper_eps}" upper="0.85" effort="50" velocity="2" />
       <mimic joint="${prefix}drive_joint" multiplier="1" offset="0" />
     </joint>
@@ -114,5 +124,5 @@
       <child link="${prefix}left_inner_knuckle" />
       <axis xyz="1 0 0" />
-      <limit lower="0" upper="0.85" effort="50" velocity="2" />
+      <limit lower="${gripper_eps}" upper="0.85" effort="50" velocity="2" />
       <mimic joint="${prefix}drive_joint" multiplier="1" offset="0" />
     </joint>
@@ -140,5 +150,5 @@
       <child link="${prefix}right_outer_knuckle" />
       <axis xyz="-1 0 0" />
-      <limit lower="0" upper="0.85" effort="50" velocity="2" />
+      <limit lower="${gripper_eps}" upper="0.85" effort="50" velocity="2" />
       <mimic joint="${prefix}drive_joint" multiplier="1" offset="0" />
     </joint>
@@ -166,5 +176,5 @@
       <child link="${prefix}right_finger" />
       <axis xyz="1 0 0" />
-      <limit lower="0" upper="0.85" effort="50" velocity="2" />
+      <limit lower="${gripper_eps}" upper="0.85" effort="50" velocity="2" />
       <mimic joint="${prefix}drive_joint" multiplier="1" offset="0" />
     </joint>
@@ -192,5 +202,5 @@
       <child link="${prefix}right_inner_knuckle" />
       <axis xyz="-1 0 0" />
-      <limit lower="0" upper="0.85" effort="50" velocity="2" />
+      <limit lower="${gripper_eps}" upper="0.85" effort="50" velocity="2" />
       <mimic joint="${prefix}drive_joint" multiplier="1" offset="0" />
     </joint>

File: xarm_moveit_config/srdf/_uf850_macro.srdf.xacro (robot description, xacro)
@@ -68,6 +68,12 @@
         <joint name="${prefix}drive_joint" />
       </group>
+      <!-- 0.02, not 0. `drive_joint`'s lower joint limit IS 0, so an "open" of exactly 0 parks the
+           jaws on a hard stop, and a physics engine does not settle exactly on a hard stop: gz left
+           the measured joint a fraction of a milliradian NEGATIVE, MoveIt/MTC judged the state out
+           of bounds, and after the first ReturnHome every later gripper MoveTo failed with "Start
+           state is out of bounds!". 0.02 rad is ~1 mm of jaw travel, so the gripper is still fully
+           open for anything the cell handles, and the joint never rests against its limit. -->
       <group_state name="open" group="${prefix}uf850_gripper">
-        <joint name="${prefix}drive_joint" value="0" />
+        <joint name="${prefix}drive_joint" value="0.02" />
       </group_state>
       <group_state name="close" group="${prefix}uf850_gripper">
