Commit message: uf850: add a distinct 'pregrasp' gripper group state
MTC's GenerateGraspPose normalises every scene it generates to the named
pre-grasp pose EXACTLY, while the arm-side interface state carries the
MEASURED joint value. Connect then drops any (start, goal) pair whose joints
outside its planned group differ by ~1e-4 — precisely the size of
gz_ros2_control's position-loop residual — so a physics-backed pick failed
intermittently to plan with "Deviation in joint drive_joint:
[0.02] != [0.020126]", every goal rejected before OMPL ran.

If the pre-grasp pose equals the pose the gripper already rests at, the task's
"open gripper" MoveTo is a no-op whose end scene keeps the measured value, and
the mismatch survives. A pre-grasp the gripper is never already at forces a
real motion, whose end scene is the exact goal, so both sides of the Connect
are exact and the deviation is structurally zero.

0.05 rad is ~3 mm wider than the resting 'open' (0.02). Everything that
releases still targets 'open', which keeps the invariant true.

Co-Authored-By: Claude Opus 5 (1M context) <noreply@anthropic.com>

File: xarm_moveit_config/srdf/_uf850_macro.srdf.xacro (robot description, xacro)
@@ -76,4 +76,17 @@
       <group_state name="open" group="${prefix}uf850_gripper">
         <joint name="${prefix}drive_joint" value="0.02" />
+      </group_state>
+      <!-- PREGRASP is deliberately a DIFFERENT value from 'open' (0.05 vs 0.02, ~3 mm wider jaws).
+           MTC's GenerateGraspPose normalises its generated scenes to this named pose EXACTLY, while
+           the arm-side interface state carries the MEASURED joint value; Connect then rejects the
+           pair if they differ by ~1e-4, which is exactly the size of gz's position-loop residual.
+           If the pre-grasp equalled the pose the gripper is already resting at, the task's "open
+           gripper" MoveTo would be a no-op whose end scene keeps the measured value and the mismatch
+           survives. Commanding a pose the gripper is never already at forces a real motion, whose
+           end scene IS the exact goal — so both sides of the Connect are exact and the deviation is
+           structurally zero. Everything that RELEASES (Place, Recover, ReturnHome) still targets
+           'open', so the gripper always rests at 0.02 and this is always a real move. -->
+      <group_state name="pregrasp" group="${prefix}uf850_gripper">
+        <joint name="${prefix}drive_joint" value="0.05" />
       </group_state>
       <group_state name="close" group="${prefix}uf850_gripper">
